File: MoP_Charging.kicad_sch (KiCad schematic)
At the start: 74 parts

Commit message: Finished schematics
Parts:
- gave numbers to parts that had none: 16
Other:
- note added: "Can be left open for f_{s} = 800kHz"
- note removed: "Can be left open for f_(s) = 800kHz"
Changed lines of the file:
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@@
 		)
 	)
-	(text "Can be left open for\nf_(s) = 800kHz"
+	(text "Can be left open for\nf_{s} = 800kHz"
 		(exclude_from_sim no)
 		(at 99.06 86.36 0)
@@
 		(on_board yes)
 		(dnp no)
-		(property "Reference" "Q?"
+		(property "Reference" "Q1401"
 			(at 134.62 59.69 90)
 			(effects
@@
 			(project "MoP_PBRD_PowerIn"
 				(path "/4d76798e-9a11-4d8d-a723-72f274a89091/4d057ef5-80c0-465a-b107-65508e007bbf/e5907f32-472c-4482-9109-9908b225fa99"
-					(reference "Q?")
+					(reference "Q1401")
 					(unit 1)
 				)
@@
 		(on_board yes)
 		(dnp no)
-		(property "Reference" "C?"
+		(property "Reference" "C1401"
 			(at 113.03 72.39 0)
 			(effects
@@
 			(project "MoP_PBRD_PowerIn"
 				(path "/4d76798e-9a11-4d8d-a723-72f274a89091/4d057ef5-80c0-465a-b107-65508e007bbf/e5907f32-472c-4482-9109-9908b225fa99"
-					(reference "C?")
+					(reference "C1401")
 					(unit 1)
 				)
@@
 		(dnp no)
 		(fields_autoplaced yes)
-		(property "Reference" "R?"
+		(property "Reference" "R1404"
 			(at 88.9 58.42 90)
 			(effects
@@
 			(project "MoP_PBRD_PowerIn"
 				(path "/4d76798e-9a11-4d8d-a723-72f274a89091/4d057ef5-80c0-465a-b107-65508e007bbf/e5907f32-472c-4482-9109-9908b225fa99"
-					(reference "R?")
+					(reference "R1404")
 					(unit 1)
 				)
@@
 		(dnp no)
 		(fields_autoplaced yes)
-		(property "Reference" "J?"
+		(property "Reference" "J1401"
 			(at 22.86 25.4 0)
 			(effects
@@
 			(project "MoP_PBRD_PowerIn"
 				(path "/4d76798e-9a11-4d8d-a723-72f274a89091/4d057ef5-80c0-465a-b107-65508e007bbf/e5907f32-472c-4482-9109-9908b225fa99"
-					(reference "J?")
+					(reference "J1401")
 					(unit 1)
 				)
@@
 		(dnp no)
 		(fields_autoplaced yes)
-		(property "Reference" "J?"
+		(property "Reference" "J1402"
 			(at 50.8 25.4 0)
 			(effects
@@
 			(project "MoP_PBRD_PowerIn"
 				(path "/4d76798e-9a11-4d8d-a723-72f274a89091/4d057ef5-80c0-465a-b107-65508e007bbf/e5907f32-472c-4482-9109-9908b225fa99"
-					(reference "J?")
+					(reference "J1402")
 					(unit 1)
 				)
@@
 		(on_board yes)
 		(dnp no)
-		(property "Reference" "Q?"
+		(property "Reference" "Q1402"
 			(at 154.94 76.2 90)
 			(effects
@@
 			(project "MoP_PBRD_PowerIn"
 				(path "/4d76798e-9a11-4d8d-a723-72f274a89091/4d057ef5-80c0-465a-b107-65508e007bbf/e5907f32-472c-4482-9109-9908b225fa99"
-					(reference "Q?")
+					(reference "Q1402")
 					(unit 1)
 				)
@@
 		(on_board yes)
 		(dnp no)
-		(property "Reference" "D?"
+		(property "Reference" "D1401"
 			(at 121.92 33.02 90)
 			(effects
@@
 			(project "MoP_PBRD_PowerIn"
 				(path "/4d76798e-9a11-4d8d-a723-72f274a89091/4d057ef5-80c0-465a-b107-65508e007bbf/e5907f32-472c-4482-9109-9908b225fa99"
-					(reference "D?")
+					(reference "D1401")
 					(unit 1)
 				)
@@
 		(dnp no)
 		(fields_autoplaced yes)
-		(property "Reference" "J?"
+		(property "Reference" "J1404"
 			(at 26.67 60.96 0)
 			(effects
@@
 			(project "MoP_PBRD_PowerIn"
 				(path "/4d76798e-9a11-4d8d-a723-72f274a89091/4d057ef5-80c0-465a-b107-65508e007bbf/e5907f32-472c-4482-9109-9908b225fa99"
-					(reference "J?")
+					(reference "J1404")
 					(unit 1)
 				)
@@
 		(dnp no)
 		(fields_autoplaced yes)
-		(property "Reference" "R?"
-			(at 82.55 69.85 0)
+		(property "Reference" "R1405"
+			(at 82.55 69.8499 0)
 			(effects
 				(font
@@
 		)
 		(property "Value" "4.99"
-			(at 82.55 72.39 0)
+			(at 82.55 72.3899 0)
 			(effects
 				(font
@@
 			(project "MoP_PBRD_PowerIn"
 				(path "/4d76798e-9a11-4d8d-a723-72f274a89091/4d057ef5-80c0-465a-b107-65508e007bbf/e5907f32-472c-4482-9109-9908b225fa99"
-					(reference "R?")
+					(reference "R1405")
 					(unit 1)
 				)
@@
 		(dnp no)
 		(fields_autoplaced yes)
-		(property "Reference" "R?"
-			(at 50.8 91.44 0)
+		(property "Reference" "R1403"
+			(at 50.8 91.4399 0)
 			(effects
 				(font
@@
 		)
 		(property "Value" "5.1k"
-			(at 50.8 93.98 0)
+			(at 50.8 93.9799 0)
 			(effects
 				(font
@@
 			(project "MoP_PBRD_PowerIn"
 				(path "/4d76798e-9a11-4d8d-a723-72f274a89091/4d057ef5-80c0-465a-b107-65508e007bbf/e5907f32-472c-4482-9109-9908b225fa99"
-					(reference "R?")
+					(reference "R1403")
 					(unit 1)
 				)
@@
 		(dnp no)
 		(fields_autoplaced yes)
-		(property "Reference" "R?"
-			(at 99.06 69.85 0)
+		(property "Reference" "R1406"
+			(at 99.06 69.8499 0)
 			(effects
 				(font
@@
 		)
 		(property "Value" "4.99"
-			(at 99.06 72.39 0)
+			(at 99.06 72.3899 0)
 			(effects
 				(font
@@
 			(project "MoP_PBRD_PowerIn"
 				(path "/4d76798e-9a11-4d8d-a723-72f274a89091/4d057ef5-80c0-465a-b107-65508e007bbf/e5907f32-472c-4482-9109-9908b225fa99"
-					(reference "R?")
+					(reference "R1406")
 					(unit 1)
 				)
@@
 		(on_board yes)
 		(dnp no)
-		(property "Reference" "C?"
+		(property "Reference" "C1402"
 			(at 125.73 72.39 0)
 			(effects
@@
 			(project "MoP_PBRD_PowerIn"
 				(path "/4d76798e-9a11-4d8d-a723-72f274a89091/4d057ef5-80c0-465a-b107-65508e007bbf/e5907f32-472c-4482-9109-9908b225fa99"
-					(reference "C?")
+					(reference "C1402")
 					(unit 1)
 				)
@@
 		(on_board yes)
 		(dnp no)
-		(property "Reference" "D?"
+		(property "Reference" "D1401"
 			(at 55.88 40.64 90)
 			(effects
@@
 			(project "MoP_PBRD_PowerIn"
 				(path "/4d76798e-9a11-4d8d-a723-72f274a89091/4d057ef5-80c0-465a-b107-65508e007bbf/e5907f32-472c-4482-9109-9908b225fa99"
-					(reference "D?")
+					(reference "D1401")
 					(unit 1)
 				)
@@
 		(on_board yes)
 		(dnp no)
-		(property "Reference" "R?"
+		(property "Reference" "R1402"
 			(at 38.1 91.44 0)
 			(effects
@@
 			(project "MoP_PBRD_PowerIn"
 				(path "/4d76798e-9a11-4d8d-a723-72f274a89091/4d057ef5-80c0-465a-b107-65508e007bbf/e5907f32-472c-4482-9109-9908b225fa99"
-					(reference "R?")
+					(reference "R1402")
 					(unit 1)
 				)
@@
 		(on_board yes)
 		(dnp no)
-		(property "Reference" "J?"
+		(property "Reference" "J1403"
 			(at 21.59 48.26 0)
 			(effects
@@
 			(project "MoP_PBRD_PowerIn"
 				(path "/4d76798e-9a11-4d8d-a723-72f274a89091/4d057ef5-80c0-465a-b107-65508e007bbf/e5907f32-472c-4482-9109-9908b225fa99"
-					(reference "J?")
+					(reference "J1403")
 					(unit 1)
 				)
@@
 		(on_board yes)
 		(dnp no)
-		(property "Reference" "U?"
-			(at 97.79 29.21 0)
+		(property "Reference" "U1401"
+			(at 99.822 29.21 0)
 			(effects
 				(font
@@
 			(project "MoP_PBRD_PowerIn"
 				(path "/4d76798e-9a11-4d8d-a723-72f274a89091/4d057ef5-80c0-465a-b107-65508e007bbf/e5907f32-472c-4482-9109-9908b225fa99"
-					(reference "U?")
+					(reference "U1401")
 					(unit 1)
 				)
@@
 		(on_board yes)
 		(dnp no)
-		(property "Reference" "R?"
+		(property "Reference" "R1401"
 			(at 109.22 25.4 90)
 			(effects
@@
 			(project "MoP_PBRD_PowerIn"
 				(path "/4d76798e-9a11-4d8d-a723-72f274a89091/4d057ef5-80c0-465a-b107-65508e007bbf/e5907f32-472c-4482-9109-9908b225fa99"
-					(reference "R?")
+					(reference "R1401")
 					(unit 1)
 				)
