File: MoP_USB-C.kicad_sch (KiCad schematic)
At the start: 14 parts, among them J501 USB4105-GF-A, U502 FT230XS

Commit message: added OBC
Changed lines of the file:
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@@
 				)
 			)
-		)
-	)
-	(symbol
-		(lib_id "power:+3V3")
-		(at 120.65 52.07 0)
-		(unit 1)
-		(exclude_from_sim no)
-		(in_bom yes)
-		(on_board yes)
-		(dnp no)
-		(fields_autoplaced yes)
-		(property "Reference" "#PWR026"
-			(at 120.65 55.88 0)
-			(effects
-				(font
-					(size 1.27 1.27)
-				)
-				(hide yes)
-			)
-		)
-		(property "Value" "R3V3"
-			(at 120.65 46.99 0)
-			(effects
-				(font
-					(size 1.27 1.27)
-				)
-			)
-		)
-		(property "Footprint" ""
-			(at 120.65 52.07 0)
-			(effects
-				(font
-					(size 1.27 1.27)
-				)
-				(hide yes)
-			)
-		)
-		(property "Datasheet" ""
-			(at 120.65 52.07 0)
-			(effects
-				(font
-					(size 1.27 1.27)
-				)
-				(hide yes)
-			)
-		)
-		(property "Description" "Power symbol creates a global label with name \"+3V3\""
-			(at 120.65 52.07 0)
-			(effects
-				(font
-					(size 1.27 1.27)
-				)
-				(hide yes)
-			)
-		)
-		(pin "1"
-		)
-		(instances
 			(project ""
-				(path "/4d76798e-9a11-4d8d-a723-72f274a89091/63f46eb8-407d-4e29-86cd-16d2149e2636"
-					(reference "#PWR026")
+				(path "/4fa4f4fb-851d-4975-b789-eb7f900188ea/6a65851d-78bc-4f90-bc40-f85ce185b9c5"
+					(reference "D1001")
 					(unit 1)
 				)
@@
 				)
 			)
+			(project "MoP"
+				(path "/4fa4f4fb-851d-4975-b789-eb7f900188ea/6a65851d-78bc-4f90-bc40-f85ce185b9c5"
+					(reference "JP1002")
+					(unit 1)
+				)
+			)
 		)
 	)
@@
 				)
 			)
+			(project ""
+				(path "/4fa4f4fb-851d-4975-b789-eb7f900188ea/6a65851d-78bc-4f90-bc40-f85ce185b9c5"
+					(reference "J1001")
+					(unit 1)
+				)
+			)
 		)
 	)
@@
 		(on_board yes)
 		(dnp no)
-		(fields_autoplaced yes)
 		(property "Reference" "R503"
-			(at 64.77 115.5699 0)
+			(at 63.754 115.57 0)
 			(effects
 				(font
@@
 				(path "/4d76798e-9a11-4d8d-a723-72f274a89091/63f46eb8-407d-4e29-86cd-16d2149e2636"
 					(reference "R503")
+					(unit 1)
+				)
+			)
+			(project "MoP"
+				(path "/4fa4f4fb-851d-4975-b789-eb7f900188ea/6a65851d-78bc-4f90-bc40-f85ce185b9c5"
+					(reference "R1003")
 					(unit 1)
 				)
@@
 				)
 			)
+			(project "MoP"
+				(path "/4fa4f4fb-851d-4975-b789-eb7f900188ea/6a65851d-78bc-4f90-bc40-f85ce185b9c5"
+					(reference "#PWR018")
+					(unit 1)
+				)
+			)
 		)
 	)
 	(symbol
-		(lib_id "power:+3V3")
-		(at 111.76 52.07 0)
+		(lib_id "power:+5V")
+		(at 120.65 52.07 0)
 		(unit 1)
 		(exclude_from_sim no)
@@
 		(dnp no)
 		(fields_autoplaced yes)
-		(property "Reference" "#PWR027"
-			(at 111.76 55.88 0)
-			(effects
-				(font
-					(size 1.27 1.27)
-				)
-				(hide yes)
-			)
-		)
-		(property "Value" "R5V"
-			(at 111.76 46.99 0)
+		(property "Reference" "#PWR01002"
+			(at 120.65 55.88 0)
+			(effects
+				(font
+					(size 1.27 1.27)
+				)
+				(hide yes)
+			)
+		)
+		(property "Value" "R3V3"
+			(at 120.65 46.99 0)
 			(effects
 				(font
@@
 		)
 		(property "Footprint" ""
-			(at 111.76 52.07 0)
+			(at 120.65 52.07 0)
 			(effects
 				(font
@@
 		)
 		(property "Datasheet" ""
-			(at 111.76 52.07 0)
-			(effects
-				(font
-					(size 1.27 1.27)
-				)
-				(hide yes)
-			)
-		)
-		(property "Description" "Power symbol creates a global label with name \"+3V3\""
-			(at 111.76 52.07 0)
+			(at 120.65 52.07 0)
+			(effects
+				(font
+					(size 1.27 1.27)
+				)
+				(hide yes)
+			)
+		)
+		(property "Description" "Power symbol creates a global label with name \"+5V\""
+			(at 120.65 52.07 0)
 			(effects
 				(font
@@
 		)
 		(instances
-			(project "MoP"
-				(path "/4d76798e-9a11-4d8d-a723-72f274a89091/63f46eb8-407d-4e29-86cd-16d2149e2636"
-					(reference "#PWR027")
+			(project "OBC"
+				(path "/4fa4f4fb-851d-4975-b789-eb7f900188ea/6a65851d-78bc-4f90-bc40-f85ce185b9c5"
+					(reference "#PWR01002")
 					(unit 1)
 				)
@@
 				)
 			)
+			(project "MoP"
+				(path "/4fa4f4fb-851d-4975-b789-eb7f900188ea/6a65851d-78bc-4f90-bc40-f85ce185b9c5"
+					(reference "JP1001")
+					(unit 1)
+				)
+			)
 		)
 	)
@@
 				(path "/4d76798e-9a11-4d8d-a723-72f274a89091/63f46eb8-407d-4e29-86cd-16d2149e2636"
 					(reference "R502")
+					(unit 1)
+				)
+			)
+			(project "MoP"
+				(path "/4fa4f4fb-851d-4975-b789-eb7f900188ea/6a65851d-78bc-4f90-bc40-f85ce185b9c5"
+					(reference "R1002")
 					(unit 1)
 				)
@@
 				)
 			)
+			(project ""
+				(path "/4fa4f4fb-851d-4975-b789-eb7f900188ea/6a65851d-78bc-4f90-bc40-f85ce185b9c5"
+					(reference "R1004")
+					(unit 1)
+				)
+			)
 		)
 	)
@@
 				(path "/4d76798e-9a11-4d8d-a723-72f274a89091/63f46eb8-407d-4e29-86cd-16d2149e2636"
 					(reference "R506")
+					(unit 1)
+				)
+			)
+			(project "MoP"
+				(path "/4fa4f4fb-851d-4975-b789-eb7f900188ea/6a65851d-78bc-4f90-bc40-f85ce185b9c5"
+					(reference "R1006")
 					(unit 1)
 				)
@@
 				)
 			)
+			(project ""
+				(path "/4fa4f4fb-851d-4975-b789-eb7f900188ea/6a65851d-78bc-4f90-bc40-f85ce185b9c5"
+					(reference "U1001")
+					(unit 1)
+				)
+			)
 		)
 	)
@@
 				)
 			)
+			(project "MoP"
+				(path "/4fa4f4fb-851d-4975-b789-eb7f900188ea/6a65851d-78bc-4f90-bc40-f85ce185b9c5"
+					(reference "D1002")
+					(unit 1)
+				)
+			)
 		)
 	)
@@
 				)
 			)
+			(project ""
+				(path "/4fa4f4fb-851d-4975-b789-eb7f900188ea/6a65851d-78bc-4f90-bc40-f85ce185b9c5"
+					(reference "R1005")
+					(unit 1)
+				)
+			)
 		)
 	)
@@
 				)
 			)
+			(project "MoP"
+				(path "/4fa4f4fb-851d-4975-b789-eb7f900188ea/6a65851d-78bc-4f90-bc40-f85ce185b9c5"
+					(reference "R1001")
+					(unit 1)
+				)
+			)
 		)
 	)
@@
 				(path "/4d76798e-9a11-4d8d-a723-72f274a89091/63f46eb8-407d-4e29-86cd-16d2149e2636"
 					(reference "C501")
+					(unit 1)
+				)
+			)
+			(project ""
+				(path "/4fa4f4fb-851d-4975-b789-eb7f900188ea/6a65851d-78bc-4f90-bc40-f85ce185b9c5"
+					(reference "C1002")
 					(unit 1)
 				)
@@
 				)
 			)
+			(project ""
+				(path "/4fa4f4fb-851d-4975-b789-eb7f900188ea/6a65851d-78bc-4f90-bc40-f85ce185b9c5"
+					(reference "#PWR016")
+					(unit 1)
+				)
+			)
+		)
+	)
+	(symbol
+		(lib_id "power:+5V")
+		(at 111.76 52.07 0)
+		(unit 1)
+		(exclude_from_sim no)
+		(in_bom yes)
+		(on_board yes)
+		(dnp no)
+		(fields_autoplaced yes)
+		(property "Reference" "#PWR01001"
+			(at 111.76 55.88 0)
+			(effects
+				(font
+					(size 1.27 1.27)
+				)
+				(hide yes)
+			)
+		)
+		(property "Value" "R5V"
+			(at 111.76 46.99 0)
+			(effects
+				(font
+					(size 1.27 1.27)
+				)
+			)
+		)
+		(property "Footprint" ""
+			(at 111.76 52.07 0)
+			(effects
+				(font
+					(size 1.27 1.27)
+				)
+				(hide yes)
+			)
+		)
+		(property "Datasheet" ""
+			(at 111.76 52.07 0)
+			(effects
+				(font
+					(size 1.27 1.27)
+				)
+				(hide yes)
+			)
+		)
+		(property "Description" "Power symbol creates a global label with name \"+5V\""
+			(at 111.76 52.07 0)
+			(effects
+				(font
+					(size 1.27 1.27)
+				)
+				(hide yes)
+			)
+		)
+		(pin "1"
+		)
+		(instances
+			(project "OBC"
+				(path "/4fa4f4fb-851d-4975-b789-eb7f900188ea/6a65851d-78bc-4f90-bc40-f85ce185b9c5"
+					(reference "#PWR01001")
+					(unit 1)
+				)
+			)
 		)
 	)
@@
 				(path "/4d76798e-9a11-4d8d-a723-72f274a89091/63f46eb8-407d-4e29-86cd-16d2149e2636"
 					(reference "C501")
+					(unit 1)
+				)
+			)
+			(project "MoP"
+				(path "/4fa4f4fb-851d-4975-b789-eb7f900188ea/6a65851d-78bc-4f90-bc40-f85ce185b9c5"
+					(reference "C1001")
 					(unit 1)
 				)
@@
 					(reference "#PWR017")
 					(unit 1)
+				)
+			)
+			(project "MoP"
+				(path "/4fa4f4fb-851d-4975-b789-eb7f900188ea/6a65851d-78bc-4f90-bc40-f85ce185b9c5"
+					(reference "#PWR017")
+					(unit 1)
