File: EPS/EPS.kicad_sch (KiCad schematic)
At the start: 13 parts, among them J1 Conn_01x02, J2 Conn_01x02, J3 Camera, J4 Steering, J5 1x2_Terminal, J6 1x2_Terminal, J7 Conn_02x20_Counter_Clockwise, U1 L293D, U2 L293D

Commit message: added OBC
Parts:
- removed U1: L293D, Package_SO:SO-20_12.8x7.5mm_P1.27mm, symbol Driver_Motor:L293D
- removed U2: L293D, Package_DIP:DIP-16_W7.62mm_Socket_LongPads, symbol Driver_Motor:L293D
- added U101, U102: L293DD, Nigels_Library:SOIC127P1032X265-20N, symbol Nigels_Library:L293DD
- J105: renamed from J7; footprint (none) -> Nigels_Library:PinHeader_2x20_P2.54mm_Vertical_CC
- renumbered J5 to J101, J6 to J102, J1 to J103, J2 to J104, J3 to J106, J4 to J107, JP2 to JP101, JP1 to JP102
Connections:
- net C1a: now also U102.3 (OUTPUT_1)
- net C1b: now also U102.8 (OUTPUT_2)
- net C2a: now also U102.13 (OUTPUT_3)
- net C2b: now also U102.18 (OUTPUT_4)
- net DC_Motor_L1: now also U101.2 (INPUT_1); no longer J105.16 (Pin_16)
- net DC_Motor_L2: now also U101.9 (INPUT_2); no longer J105.17 (Pin_17)
- net DC_Motor_L_EN: now also U101.1 (ENABLE_1)
- net DC_Motor_R1: now also U101.12 (INPUT_3); no longer J105.18 (Pin_18)
- net DC_Motor_R2: now also U101.19 (INPUT_4); no longer J105.19 (Pin_19)
- net DC_Motor_R_EN: now also U101.11 (ENABLE_2)
- net GND: now also U101.14 (GND__4), U101.15 (GND__5), U101.16 (GND__6), U101.17 (GND__7), U101.4 (GND), U101.5 (GND__1), U101.6 (GND__2), U101.7 (GND__3), U102.14 (GND__4), U102.15 (GND__5), U102.16 (GND__6), U102.17 (GND__7), U102.4 (GND), U102.5 (GND__1), U102.6 (GND__2), U102.7 (GND__3)
- net LDCM_Y1: now also U101.3 (OUTPUT_1)
- net LDCM_Y2: now also U101.8 (OUTPUT_2)
- net RDCM_Y1: now also U101.13 (OUTPUT_3)
- net RDCM_Y2: now also U101.18 (OUTPUT_4)
- net Stepper0: now also U102.2 (INPUT_1)
- net Stepper1: now also U102.9 (INPUT_2)
- net Stepper2: now also U102.12 (INPUT_3)
- net Stepper3: now also U102.19 (INPUT_4)
- net VCC: now also U102.1 (ENABLE_1), U102.10 (VS), U102.11 (ENABLE_2), U102.20 (VSS)
- net VS: now also U101.10 (VS), U101.20 (VSS)
- no-connect marks 16 -> 20
Other:
- company: (none) -> ESE - Conestoga
- title: (none) -> MoP - EPS
- moved on the sheet: J101, J102, J103, J104, JP101, JP102, R1, R2
